File: pcb/led-sign/led-sign.kicad_sch (KiCad schematic)
At the start: 42 parts, among them J1 USB_C_Receptacle, J2 Conn_01x03_Socket, Q1 PMOS, SW1 SW_Push, U1 nRF52832-QFxx, U2 TP4056-42-ESOP8, U3 LP5907MFX-3.3, U4 LP5024, U5 LP5024, Y1 32MHz

Commit message: start layout
Signed-off-by: 3nt3 <gott@3nt3.de>
Parts:
- removed C17, C20: 10u, symbol Device:C
- removed C18: 1u, symbol Device:C
- removed C19: 100n, symbol Device:C
- removed U4, U5: LP5024, symbol 3nt3:LP5024
- removed Y1: 32MHz, symbol Device:Crystal
- added D1, D2: LED, kicad-lib:LED_0603_1608Metric_Pad1.05x0.95mm_HandSolder_Triangle, symbol Device:LED
- added R10, R11: 1M, Resistor_SMD:R_0603_1608Metric_Pad0.98x0.95mm_HandSolder, symbol Device:R
- added R9: 10K, Resistor_SMD:R_0603_1608Metric_Pad0.98x0.95mm_HandSolder, symbol Device:R
- added SW2: SW_Push, easyeda2kicad:SW-SMD_4P-L5.1-W5.1-P3.70-LS6.5-TL_H1.5, symbol Switch:SW_Push
- added Y1: Crystal_GND24_Small, Crystal:Crystal_SMD_3225-4Pin_3.2x2.5mm, symbol Device:Crystal_GND24_Small
- AE1: footprint footprints:pcb antenna -> RF_Antenna:Texas_SWRA117D_2.4GHz_Left
- BT1: footprint (none) -> Connector_JST:JST_SH_SM02B-SRSS-TB_1x02-1MP_P1.00mm_Horizontal
- C1, C10, C11, C12, C13, C14, C15, C2, C3, C4, C5, C6, C7, C8, C9: footprint (none) -> Capacitor_SMD:C_0603_1608Metric_Pad1.08x0.95mm_HandSolder
- C16: value 1u -> 100n; footprint (none) -> Capacitor_SMD:C_0603_1608Metric_Pad1.08x0.95mm_HandSolder
- D4: footprint (none) -> Diode_SMD:D_0603_1608Metric_Pad1.05x0.95mm_HandSolder
- J1: footprint (none) -> easyeda2kicad:USB-C-SMD_MC-311D
- J2: footprint (none) -> Connector_JST:JST_SH_SM03B-SRSS-TB_1x03-1MP_P1.00mm_Horizontal
- L1: footprint (none) -> Inductor_SMD:L_0603_1608Metric_Pad1.05x0.95mm_HandSolder
- Q1: footprint (none) -> Package_TO_SOT_SMD:SOT-23_Handsoldering
- R1, R2, R3, R4, R5, R6, R7, R8: footprint (none) -> Resistor_SMD:R_0603_1608Metric_Pad0.98x0.95mm_HandSolder
- SW1: footprint (none) -> easyeda2kicad:SW-SMD_4P-L5.1-W5.1-P3.70-LS6.5-TL_H1.5
Connections:
- net +3V3: now also R9.1
- net GND: now also C6.2, R11.2, SW2.2; no longer C6.1
- net I2C_EN: now also U1.8 (P0.06)
- net I2C_SCL: now also U1.9 (P0.07)
- net I2C_SDA: now also U1.10 (P0.08)
- net at C16.1: now also U1.4 (P0.02/AIN0), R10.2, R11.1
- net VBAT: now reaches BT1.1 (+), C1.1, Q1.1 (D), U2.5 (BAT)
- net VBAT: now also R10.1
- net at C5.2: now also Y1.4; no longer U1.34 (XC1)
- net USER_BUTTON: now reaches C15.1
- net USER_BUTTON: now also U1.14 (P0.11), R9.2, SW2.1
- net at U2.6 (~{STDBY}): now also D2.1 (K)
- net at U2.7 (~{CHRG}): now also D1.1 (K)
- net at R4.2: now also D1.2 (A)
- net at R5.2: now also D2.2 (A)
- net at U1.35 (XC2): now also Y1.1; no longer C6.2
- new net: C6.1, Y1.2
- new net: U1.34 (XC1), Y1.3
Other:
- note added: "voltage divider for VBAT"
- moved on the sheet: AE1, BT1, C1, C10, C11, C12, C13, C14, C2, C3, C4, C5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
